Commit message: coffee_cup blend and urdf and other file updates. trying to find good box for coffee_cup, 50 tea cups experiment

File: data/coffee_cup.urdf (robot description, URDF)
Before this commit: robot TeaCup, 1 links, 0 joints
Links:
- link TeaCupLink: geometry collision box size=0.2 0.2 0.2; visual mesh filename=coffee_cup.obj scale=0.1 0.1 0.1

Commit message: Modified models

File: data/coffee_cup.urdf (robot description, URDF)
Before this commit: robot TeaCup, 1 links, 0 joints
Links:
- link TeaCupLink: geometry collision cylinder length=15 radius=6; visual mesh filename=coffee_cup.obj scale=1.0 1.0 1.0
