Commit message: Crazy mad shit with vector urdf+sdf to create awesome gif of two teams of vectors fighting with cups falling on them. Fixed tea cup collider with cylinder

File: data/TeaCup.urdf (robot description, URDF)
Before this commit: robot TeaCup, 1 links, 0 joints
Links:
- link TeaCupLink: mass None -> 0.5; geometry collision cylinder length=2.816 radius=1.0; visual mesh filename=TeaCup.obj
