Commit message: Updated urdf of vector and moved wheel joints into correct place (changed a million origins, removed poses). Added head.mtl and texture uv map (because pybullet can only use 1 material per obj...)

File: data/vector_from_sdf.urdf (robot description, URDF)
Before this commit: robot Vector, 8 links, 0 joints
Links:
- removed link anki_vector::anki_vector::robot::body
- added link body, mass 0.8; collision box size=0.065 0.045 0.07; visual mesh filename=body.obj scale=0.01 0.01 0.01
- link anki_vector::anki_vector::robot::tracks: geometry collision box size=0.072 0.055 0.06; visual mesh filename=tracks.obj scale=0.01 0.01 0.01
Joints:
- added joint anki_vector::anki_vector::robot::forklift: type fixed, parent body, child anki_vector::anki_vector::robot::forklift
- added joint anki_vector::anki_vector::robot::head_tilt: type fixed, parent body, child anki_vector::anki_vector::robot::head
- added joint anki_vector::anki_vector::robot::tracks: type fixed, parent body, child anki_vector::anki_vector::robot::tracks
- added joint anki_vector::anki_vector::robot::wheel_BL_hinge: type revolute, parent body, child anki_vector::anki_vector::robot::wheel_BL, origin xyz=-0.045 0.022 0.0105 rpy=0 -0 0, axis 0 1 0, limit lower=-1e+16 upper=1e+16 effort=-1 velocity=-1
- added joint anki_vector::anki_vector::robot::wheel_BR_hinge: type revolute, parent body, child anki_vector::anki_vector::robot::wheel_BR, origin xyz=-0.045 -0.022 0.0105 rpy=0 -0 0, axis 0 1 0, limit lower=-1e+16 upper=1e+16 effort=-1 velocity=-1
- added joint anki_vector::anki_vector::robot::wheel_FL_hinge: type revolute, parent body, child anki_vector::anki_vector::robot::wheel_FL, origin xyz=-0.003 0.022 0.014 rpy=0 -0 0, axis 0 1 0, limit lower=-1e+16 upper=1e+16 effort=-1 velocity=-1
- added joint anki_vector::anki_vector::robot::wheel_FR_hinge: type revolute, parent body, child anki_vector::anki_vector::robot::wheel_FR, origin xyz=-0.003 -0.022 0.014 rpy=0 -0 0, axis 0 1 0, limit lower=-1e+16 upper=1e+16 effort=-1 velocity=-1

Commit message: Got FPS view from vector in env. Changed wheel position a bit but suspicious.

File: data/vector_from_sdf.urdf (robot description, URDF)
Before this commit: robot Vector, 8 links, 7 joints
Joints:
- joint anki_vector::anki_vector::robot::wheel_FL_hinge: origin xyz=-0.003 0.022 0.014 rpy=0 -0 0 -> xyz=0.003 0.022 0.014 rpy=0 -0 0
- joint anki_vector::anki_vector::robot::wheel_FR_hinge: origin xyz=-0.003 -0.022 0.014 rpy=0 -0 0 -> xyz=0.003 -0.022 0.014 rpy=0 -0 0
