Commit message: Added tissue box, chips, banana, beer bottle, knife, door to kitchen walls. Updated fork, table, spoon and glass urdf.

File: data/fork.urdf (robot description, URDF)
Before this commit: robot fork, 1 links, 0 joints
Links:
- link fork: geometry collision mesh filename=fork.stl; visual mesh filename=fork.stl

File: data/glass.urdf (robot description, URDF)
Before this commit: robot glass, 1 links, 0 joints
Links:
- link base_link: mass None -> 0.5

File: data/kitchen_walls.urdf (robot description, URDF)
Before this commit: robot walls, 8 links, 7 joints
Links:
- link door_between_kitchen_and_living_room: mass 1 -> None; geometry collision mesh filename=Door.obj scale=0.01 0.01 0.01; visual mesh filename=Door.obj scale=0.01 0.01 0.01
- link wall_between_kitchen_and_living_room_1: geometry collision box size=0.15 2 1.5; visual box size=0.15 1.75 1.5
- link wall_between_kitchen_and_living_room_2: geometry collision box size=0.15 1.6 1.5; visual box size=0.15 1.6 1.5
Joints:
- joint door_to_wall_joint: origin xyz=1.5 4.5 0.75 -> xyz=1.75 4.5 0.75

File: data/spoon.urdf (robot description, URDF)
Before this commit: robot spoon, 1 links, 0 joints
Links:
- link spoon: geometry collision mesh filename=spoon.dae.obj; visual mesh filename=spoon.dae.obj

File: data/table.urdf (robot description, URDF)
Before this commit: robot none, 1 links, 0 joints
Links:
- link none: geometry collision box size=1.000000 0.535714 0.4; visual mesh filename=table4.obj
