Commit message: Updated bed, lamp, added floor

File: data/kitchen_walls.urdf (robot description, URDF)
Before this commit: robot walls, 7 links, 6 joints
Links:
- added link floor, mass 0; collision box size=4.4 10 0.2; visual box size=4.4 10 0.2
Joints:
- added joint left_to_floor: type fixed, parent floor, child left_wall

Commit message: Put all objects into config list to loop through, stored unique names and created dict. subplots, grid-class datastructure list of lists. legend and grid colours not matched, debugging code. Raised wall height to door height.

File: data/kitchen_walls.urdf (robot description, URDF)
Before this commit: robot walls, 8 links, 7 joints
Links:
- link bottom_wall: geometry collision box size=0.15 4.5 2.25; visual box size=0.15 4.5 2.25
- link floor: geometry collision box size=4.3 10 0.2; visual box size=4.3 10 0.2
- link left_wall: geometry collision box size=0.15 10 2.25; visual box size=0.15 10 2.25
- link right_wall: geometry collision box size=0.15 10 2.25; visual box size=0.15 10 2.25
- link top_wall: geometry collision box size=0.15 4.5 2.25; visual box size=0.15 4.5 2.25
- link wall_between_kitchen_and_living_room_1: geometry collision box size=0.15 2 2.25; visual box size=0.15 1.75 2.25
- link wall_between_kitchen_and_living_room_2: geometry collision box size=0.15 1.6 2.25; visual box size=0.15 1.6 2.25
